File: Hardware/MainBoard_V1.brd (EAGLE design)
At the start: 85 x 50 mm, 25 parts, among them IC1 REG1117, J1 NANO_FOOTPRINTNANO, J4 I2C, K1 RELAY-SPDT-JZC-11F, Q2 600mA/40V, Q3 600mA/40V, U1 MOC3021M, U2 TXB0104, U4 MCT2EM, X2 AC

Commit message: Bug fix
Connections:
- net D3: now also U4.5; no longer U4.6
Routing:
- net D3: track 61.5 -> 59.5 mm
Changed lines of the file:
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@@
 <drawing>
 <settings>
-<setting alwaysvectorfont="yes"/>
+<setting alwaysvectorfont="no"/>
 <setting verticaltext="up"/>
 </settings>
@@
 <contactref element="J2" pad="6"/>
 <wire x1="2.54" y1="26.67" x2="5.65" y2="27.27" width="0.6096" layer="16"/>
-<contactref element="U4" pad="6"/>
 <contactref element="R4" pad="1"/>
 <via x="11.938" y="34.036" extent="1-16" drill="0.35"/>
@@
 <via x="30.734" y="37.846" extent="1-16" drill="0.35"/>
 <wire x1="30.734" y1="37.846" x2="31.2332" y2="37.3468" width="0.4064" layer="16"/>
-<wire x1="31.2332" y1="37.3468" x2="31.2332" y2="30.84915625" width="0.4064" layer="16"/>
-<wire x1="31.2332" y1="30.84915625" x2="34.62235625" y2="27.46" width="0.4064" layer="16"/>
-<wire x1="34.62235625" y1="27.46" x2="36.19" y2="27.46" width="0.4064" layer="16"/>
+<wire x1="31.2332" y1="37.3468" x2="31.2332" y2="32.62715625" width="0.4064" layer="16"/>
 <wire x1="29.468" y1="37.511" x2="29.511" y2="37.511" width="0.4064" layer="1"/>
 <wire x1="29.511" y1="37.511" x2="30.29" y2="38.29" width="0.4064" layer="1"/>
+<contactref element="U4" pad="5"/>
+<wire x1="36.19" y1="30" x2="33.86035625" y2="30" width="0.4064" layer="16"/>
+<wire x1="33.86035625" y1="30" x2="31.2332" y2="32.62715625" width="0.4064" layer="16"/>
 </signal>
 <signal name="D4">
