File: Hardware/GaggiaBoard_V2/EAGLE/GaggiaBoard_V2.sch (EAGLE design)
At the start: 115 parts, among them IC1 LD117AS33TR, J1 4PIN, J11 PIN262409-1, J12 PIN262409-1, J13 PIN262409-1, J14 PIN262409-1, J15 PIN262409-1, J16 PIN262409-1, J17 PIN262409-1, J18 PIN262409-1, J19 PIN262409-1, J2 Vertical Qwiic Connector, J20 PIN262409-1, J3 Vertical Qwiic Connector, J5 2PIN, J6 3PIN, J7 3PIN, J8 5PIN, J9 3PIN, K1 RELAY-SPDT-JZC-11F, K2 RELAY-SPDT-JZC-11F, K3 AQH213, Q1 600mA/40V, Q10 600mA/40V, Q11 MOSFET_PCH_DUAL-DMP2240UDM, Q2 600mA/40V, Q3 600mA/40V, Q4 600mA/40V, Q5 600mA/40V, Q6 600mA/40V, Q8 600mA/40V, Q9 600mA/40V, U1 BLACKPILL, U2 MAX31855K, U5 TXS0102

Commit message: pull downs on GPIO outputs
Parts:
- added R36, R37, R38, R39, R40, R41: 3K3, rcl:R-US_R0603
Connections:
- net GND: now also R36.1, R37.1, R38.1, R39.1, R40.1, R41.1
- net PA15: now also R37.2
- net PA8: now also R36.2
- net PB12: now also R40.2
- net PB13: now also R39.2
- net PB14: now also R41.2
- net PC13: now also R38.2
Other:
- moved on the sheet: Q11G$1, Q12Q1, R32, R34
