File: Hardware/GaggiaBoard_V3/EAGLE/GaggiaBoard_V3.brd (EAGLE design)
At the start: 45 x 100 mm, 78 parts, among them IC1 LD117AS33TR, J1 4PIN, J10 PIN262409-1, J11 PIN262409-1, J12 PIN262409-1, J13 PIN262409-1, J2 Vertical Qwiic Connector, J27 6PIN, J5 2PIN, J6 3PIN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

Commit message: Snubber change
Connections:
- net AC_N: no longer C16.1, C5.1
- net AC_P: now also C16.1, C5.1
Routing:
- net AC_P: track 101.7 -> 111.4 mm
- net AC_N: track 38.8 -> 29.2 mm
- net N$9: track 19.7 -> 23.3 mm, vias 2 -> 4
Changed lines of the file:
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@@
 <drawing>
 <settings>
-<setting alwaysvectorfont="yes"/>
+<setting alwaysvectorfont="no"/>
 <setting verticaltext="up"/>
 </settings>
-<grid distance="1" unitdist="mm" unit="mm" style="lines" multiple="1" display="no" altdistance="0.1" altunitdist="mm" altunit="mm"/>
+<grid distance="50" unitdist="mil" unit="mil" style="lines" multiple="1" display="no" altdistance="5" altunitdist="mil" altunit="mil"/>
 <layers>
 <layer number="1" name="Top" color="4" fill="1" visible="yes" active="yes"/>
@@
 <class number="0" name="default" width="0" drill="0">
 </class>
+<class number="1" name="TC" width="0" drill="0">
+<clearance class="1" value="0.508"/>
+</class>
+<class number="2" name="Analog" width="0" drill="0">
+<clearance class="2" value="0.254"/>
+</class>
 </classes>
 <designrules name="default *">
@@
 <wire x1="30" y1="38.15" x2="31.15" y2="38.15" width="0.254" layer="16"/>
 <wire x1="31.15" y1="38.15" x2="32" y2="39" width="0.254" layer="16"/>
-<polygon width="0.1524" layer="1" pour="cutout">
-<vertex x="4" y="88"/>
-<vertex x="10.5" y="88"/>
-<vertex x="10.5" y="84.7"/>
-<vertex x="4" y="84.7"/>
-</polygon>
-<polygon width="0.1524" layer="16" pour="cutout">
-<vertex x="2.5" y="88"/>
-<vertex x="12" y="88"/>
-<vertex x="12" y="83"/>
-<vertex x="9" y="80"/>
-<vertex x="5.5" y="80"/>
-<vertex x="2.5" y="83"/>
-</polygon>
-<polygon width="0.1524" layer="16" pour="cutout">
-<vertex x="39" y="94"/>
-<vertex x="41" y="94"/>
-<vertex x="41" y="90.3"/>
-<vertex x="39" y="90.3"/>
-</polygon>
-<polygon width="0.1524" layer="1" pour="cutout">
-<vertex x="39" y="94"/>
-<vertex x="41" y="94"/>
-<vertex x="41" y="92"/>
-<vertex x="39" y="92"/>
-</polygon>
 </signal>
 <signal name="5V">
@@
 <contactref element="U1" pad="P2$6"/>
 </signal>
-<signal name="N$5">
+<signal name="N$5" class="1">
 <contactref element="FB2" pad="2"/>
 <contactref element="U2" pad="2"/>
@@
 <wire x1="6.865" y1="83.785" x2="6.65" y2="84" width="0.508" layer="16"/>
 </signal>
-<signal name="N$26">
+<signal name="N$26" class="1">
 <contactref element="FB1" pad="2"/>
 <contactref element="U2" pad="3"/>
@@
 <wire x1="8.135" y1="83.785" x2="8.35" y2="84" width="0.508" layer="16"/>
 </signal>
-<signal name="PRESSURE">
+<signal name="PRESSURE" class="2">
 <contactref element="J6" pad="3"/>
 <contactref element="U4" pad="4"/>
@@
 <wire x1="21" y1="77.85" x2="21" y2="79.08" width="0.254" layer="16"/>
 </signal>
-<signal name="N$3">
+<signal name="N$3" class="1">
 <contactref element="FB2" pad="1"/>
 <contactref element="J4" pad="1"/>
@@
 <wire x1="5.05" y1="85.85" x2="5.5" y2="86.3" width="0.508" layer="16"/>
 </signal>
-<signal name="N$4">
+<signal name="N$4" class="1">
 <contactref element="FB1" pad="1"/>
 <contactref element="J4" pad="2"/>
@@
 <wire x1="6.46" y1="5" x2="11.54" y2="5" width="2.54" layer="16"/>
 <wire x1="28.5" y1="3.75" x2="27.25" y2="5" width="1.27" layer="16"/>
-<wire x1="27.25" y1="5" x2="25.019" y2="5" width="1.27" layer="16"/>
-<contactref element="C5" pad="1"/>
-<contactref element="C16" pad="1"/>
-<wire x1="25.019" y1="5" x2="11.54" y2="5" width="1.27" layer="16"/>
-<wire x1="25" y1="11.6" x2="25" y2="5.019" width="1.27" layer="16"/>
-<wire x1="25" y1="5.019" x2="25.019" y2="5" width="1.27" layer="16"/>
-<wire x1="28" y1="11.6" x2="25" y2="11.6" width="1.27" layer="16"/>
+<wire x1="11.54" y1="5" x2="27.25" y2="5" width="1.27" layer="16"/>
 </signal>
 <signal name="AC_P">
@@
 <wire x1="6.509871875" y1="32.101971875" x2="4.8879" y2="30.48" width="0.508" layer="1"/>
 <wire x1="6.46" y1="10" x2="11.54" y2="10" width="1.27" layer="1"/>
+<contactref element="C5" pad="1"/>
+<contactref element="C16" pad="1"/>
+<wire x1="28" y1="11.6" x2="25" y2="11.6" width="1.27" layer="16"/>
+<wire x1="25" y1="11.6" x2="23.301" y2="9.901" width="1.27" layer="16"/>
+<wire x1="23.301" y1="9.901" x2="19" y2="9.901" width="1.27" layer="16"/>
 </signal>
 <signal name="3WAY">
@@
 <via x="12" y="26" extent="1-16" drill="0.35"/>
 <via x="22" y="14" extent="1-16" drill="0.35"/>
-<wire x1="22" y1="16" x2="22" y2="14" width="0.508" layer="1"/>
-<wire x1="22" y1="16" x2="12" y2="26" width="0.508" layer="1"/>
 <wire x1="21.311" y1="16.099" x2="21.311" y2="14.689" width="0.3048" layer="16"/>
 <wire x1="22" y1="14" x2="21.311" y2="14.689" width="0.3048" layer="16"/>
 <wire x1="12" y1="26" x2="10.85" y2="26" width="0.508" layer="16"/>
+<via x="13" y="26" extent="1-16" drill="0.35"/>
+<via x="22" y="13" extent="1-16" drill="0.35"/>
+<wire x1="22" y1="13" x2="22" y2="14" width="0.508" layer="1"/>
+<wire x1="12" y1="26" x2="13" y2="26" width="0.508" layer="1"/>
+<wire x1="13" y1="26" x2="22" y2="17" width="0.508" layer="1"/>
+<wire x1="22" y1="17" x2="22" y2="14" width="0.508" layer="1"/>
+<wire x1="13" y1="26" x2="12" y2="26" width="0.508" layer="16"/>
+<wire x1="22" y1="13" x2="22" y2="14" width="0.508" layer="16"/>
 </signal>
 <signal name="PUMP_P">
